Commit message: edit base_joint origin
xyz ="0 0 0.090" to xzy="0 0 0"

File: urdf/moiro.xacro (robot description, xacro)
@@ -9,5 +9,5 @@
   <parent link="base_footprint"/>
   <child link="base_link" />
-  <origin xyz="0 0 0.090" rpy="0 0 0"/>
+  <origin xyz="0 0 0" rpy="0 0 0"/>
 </joint>
 <link name="base_link">
